File: main.kicad_pcb (KiCad board)
At the start: 2 copper layers, 110 x 176 mm, 110 parts, among them J1 Conn_01x02_Pin, J10 TOUCH, J11 PHOTO, J12 PHOTO, J15 Conn_01x02_Pin, J16 TOF, J17 CAMERA, J18 Conn_01x15, J2 RP2350, J5 Conn_01x04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

Commit message: Add files via upload
Parts:
- moved C20 304.2 mm to (226.1, 153.5)
- moved C23 304.2 mm to (226.1, 153.5)
- moved C24 304.2 mm to (218.6, 161.9)
- moved C28 304.2 mm to (227.4, 155.4)
- moved C30 304.2 mm to (211.4, 162.1)
- moved D3 304.2 mm to (241.6, 183.8)
- moved R25 304.2 mm to (227.6, 176.4)
- moved R28 304.2 mm to (216.8, 139.7)
- moved R4 304.2 mm to (229.6, 176.4)
- moved U3 304.2 mm to (226.1, 171.6)
- moved C1 304.2 mm to (190.2, 174.5)
- moved C15 304.2 mm to (186.5, 164.4)
- moved C21 304.2 mm to (219.4, 170.1)
- moved C26 304.2 mm to (233.2, 160.3)
- moved MD1 304.2 mm to (176.0, 163.3)
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